File: PCB/YellowAdapterPCB/YellowAdapterPCB.kicad_sch (KiCad schematic)
At the start: 1 part

Commit message: Schematic first draft
Parts:
- added C1, C2, C8: 0.1uF, Altium:0603C, symbol Device:C_Small
- added C3, C4, C5, C6, C7: 0.47uF, Altium:0603C, symbol Device:C_Small
- added IC1: PCA9671PW,118, BFH stuff:SOP65P640X110-24N, symbol PCA9671PW_118:PCA9671PW,118
- added IC2: TLA2021IRUGT, BFH stuff:ADS1018IRUGT, symbol TLA2021IRUGT:TLA2021IRUGT
- added IC3: TLA2024IRUGR, BFH stuff:ADS7142IRUGT, symbol TLA2024IRUGR:TLA2024IRUGR
- added J1: Conn_02x20_Odd_Even, Connector_PinHeader_2.54mm:PinHeader_2x20_P2.54mm_Vertical, symbol Connector_Generic:Conn_02x20_Odd_Even
- added J2: ~, Connector_PinHeader_2.54mm:PinHeader_1x07_P2.54mm_Vertical, symbol nucleoidk:7x1_pin_header
- added R1, R2, R8: 1k, Altium:0603R, symbol Device:R_US
- added R3, R4, R5, R6, R7: 100, Altium:0603R, symbol Device:R_US
Connections:
- net +3v3: now reaches BOARD1.+3v3
- net +5v: now reaches BOARD1.+5v
- net +5v: now also J1.2 (Pin_2), J1.4 (Pin_4), J2.1, J2.4
- net E5V: now reaches BOARD1.E5V
- net GND: now reaches BOARD1.GND
- net GND: now also C1.1, C2.1, C3.2, C4.2, C5.2, C6.2, C7.2, C8.1, IC1.12 (VSS), IC1.2 (AD1), IC1.21 (AD0), IC1.3 (AD2), IC2.1 (ADDR), IC2.3 (GND), IC2.5 (AIN1), IC3.3 (GND), J1.14 (Pin_14), J1.20 (Pin_20), J1.25 (Pin_25), J1.30 (Pin_30), J1.34 (Pin_34), J1.39 (Pin_39), J1.6 (Pin_6), J1.9 (Pin_9), J2.3, J2.7
- net NRST: now reaches BOARD1.NRST
- net NRST: now also J1.12 (Pin_12)
- net PA_0: now reaches BOARD1.PA_0
- net PA_0: now also R6.2
- net PA_1: now reaches BOARD1.PA_1
- net PA_1: now also R3.2
- net PA_10: now reaches BOARD1.PA_10
- net PA_10: now also J1.18 (Pin_18)
- net PA_11: now reaches BOARD1.PA_11
- net PA_12: now reaches BOARD1.PA_12
- net PA_13: now reaches BOARD1.PA_13
- net PA_14: now reaches BOARD1.PA_14
- net PA_15: now reaches BOARD1.PA_15
- net PA_15: now also J1.26 (Pin_26)
- net PA_2: now reaches BOARD1.PA_2
- net PA_3: now reaches BOARD1.PA_3
- net PA_4: now reaches BOARD1.PA_4
- net PA_4: now also R4.2
- net PA_5: now reaches BOARD1.PA_5
- net PA_5: now also J1.38 (Pin_38)
- net PA_6: now reaches BOARD1.PA_6
- net PA_6: now also J1.36 (Pin_36)
- net PA_7: now reaches BOARD1.PA_7
- net PA_7: now also IC1.16 (P13)
- net PA_8: now reaches BOARD1.PA_8
- net PA_8: now also J1.33 (Pin_33)
- net PA_9: now reaches BOARD1.PA_9
- net PA_9: now also J1.32 (Pin_32)
- net PB_0: now reaches BOARD1.PB_0
- net PB_0: now also R5.2
- net PB_1: now reaches BOARD1.PB_1
- net PB_1: now also R7.2
- net PB_10: now reaches BOARD1.PB_10
- net PB_12: now reaches BOARD1.PB_12
- net PB_12: now also IC1.15 (P12)
- net PB_13: now reaches BOARD1.PB_13
- net PB_13: now also J1.16 (Pin_16)
- net PB_14: now reaches BOARD1.PB_14
- net PB_14: now also J1.31 (Pin_31)
- net PB_15: now reaches BOARD1.PB_15
- net PB_15: now also J1.29 (Pin_29)
- net PB_2: now reaches BOARD1.PB_2
- net PB_2: now also J1.13 (Pin_13)
- net PB_3: now reaches BOARD1.PB_3
- net PB_4: now reaches BOARD1.PB_4
- net PB_5: now reaches BOARD1.PB_5
- net PB_6: now reaches BOARD1.PB_6
- net PB_6: now also J1.37 (Pin_37)
- net PB_7: now reaches BOARD1.PB_7
- net PB_7: now also J1.7 (Pin_7)
- net I2C_SCL: now reaches BOARD1.PB_8
- net I2C_SCL: now also IC1.22 (SCL), IC2.10 (SCL), IC3.10 (SCL), J1.5 (Pin_5), R1.1
- net I2C_SDA: now reaches BOARD1.PB_9
- net I2C_SDA: now also IC1.23 (SDA), IC2.9 (SDA), IC3.9 (SDA), J1.3 (Pin_3), R2.1
- net PC_0: now reaches BOARD1.PC_0
- net PC_0: now also IC1.17 (P14)
- net PC_1: now reaches BOARD1.PC_1
- net PC_1: now also IC1.8 (P04)
- net PC_10: now reaches BOARD1.PC_10
- net PC_10: now also J1.23 (Pin_23)
- net PC_11: now reaches BOARD1.PC_11
- net PC_11: now also J1.21 (Pin_21)
- net PC_12: now reaches BOARD1.PC_12
- net PC_12: now also J1.19 (Pin_19)
- net PC_13: now reaches BOARD1.PC_13
- net PC_13: now also J1.11 (Pin_11)
- net PC_14: now reaches BOARD1.PC_14
- net PC_15: now reaches BOARD1.PC_15
- net PC_2: now reaches BOARD1.PC_2
- net PC_2: now also IC1.6 (P02)
- net PC_3: now reaches BOARD1.PC_3
- net PC_3: now also IC1.7 (P03)
- net PC_4: now reaches BOARD1.PC_4
- net PC_4: now also J1.22 (Pin_22)
- net PC_5: now reaches BOARD1.PC_5
- net PC_6: now reaches BOARD1.PC_6
- net PC_6: now also IC1.14 (P11)
- net PC_7: now reaches BOARD1.PC_7
- net PC_7: now also J1.15 (Pin_15)
- net PC_8: now reaches BOARD1.PC_8
- net PC_8: now also IC1.13 (P10)
- net PC_9: now reaches BOARD1.PC_9
- net PC_9: now also IC1.18 (P15)
- net PD_2: now reaches BOARD1.PD_2
- net PD_2: now also J1.24 (Pin_24)
- net PH_0: now reaches BOARD1.PH_0
- net PH_1: now reaches BOARD1.PH_1
- net PH_1: now also IC1.5 (P01)
- net U5V: now reaches BOARD1.U5V
- new net: C6.1, IC3.4 (AIN0), R6.1
- new net: C3.1, IC3.5 (AIN1), R3.1
- new net: C4.1, IC3.6 (AIN2), R4.1
- new net: C5.1, IC3.7 (AIN3), R5.1
- new net: C7.1, IC2.4 (AIN0), R7.1
- new net Expander_Reset: IC1.1 (~{RESET}), J1.40 (Pin_40), R8.2
- new net Lidar_PWM: J1.35 (Pin_35), J2.2
- new net Lidar_RX: J1.10 (Pin_10), J2.5
- new net Lidar_TX: J1.8 (Pin_8), J2.6
- new net Pi_3v3: C1.2, C2.2, C8.2, IC1.24 (VDD), IC2.8 (VDD), IC3.1 (ADDR), IC3.8 (VDD), J1.1 (Pin_1), J1.17 (Pin_17), R1.2, R2.2, R8.1
Other:
- moved on the sheet: BOARD1
